File: Digilent Discovery LA Adapter/Digilent Discovery LA Adapter.kicad_sch (KiCad schematic)
At the start: 7 parts, among them J1 Cerberus_Expansion, J2 Card_Header, J3 Addr_Main_Data, J4 CTRL2, J4 XE_Header

Commit message: labeled DD headers in sch and updated to pcb
Parts:
- added J6: XE_LA, Connector_PinHeader_2.54mm:PinHeader_1x02_P2.54mm_Vertical, symbol Connector_Generic:Conn_01x02
- added J7: Power, Connector_PinHeader_2.54mm:PinHeader_1x02_P2.54mm_Vertical, symbol Connector_Generic:Conn_01x02
- J4: renamed from J3; value Addr_Main_Data -> Addr_Data
- renumbered J4 to J3, J4 to J5
Connections:
- net +5V: now also J7.1 (Pin_1)
- net GND: now also J6.2 (Pin_2), J7.2 (Pin_2)
- net XA0: now also J4.3 (Pin_3)
- net XA1: now also J4.4 (Pin_4)
- net XA10: now also J4.15 (Pin_15)
- net XA11: now also J4.16 (Pin_16)
- net XA12: now also J4.17 (Pin_17)
- net XA13: now also J4.18 (Pin_18)
- net XA14: now also J4.19 (Pin_19)
- net XA15: now also J4.20 (Pin_20)
- net XA2: now also J4.5 (Pin_5)
- net XA3: now also J4.6 (Pin_6)
- net XA4: now also J4.7 (Pin_7)
- net XA5: now also J4.8 (Pin_8)
- net XA6: now also J4.9 (Pin_9)
- net XA7: now also J4.10 (Pin_10)
- net XA8: now also J4.13 (Pin_13)
- net XA9: now also J4.14 (Pin_14)
- net XBUSACK: now also J5.5 (Pin_5)
- net XBUSREQ: now also J5.3 (Pin_3)
- net XCLK: now also J5.1 (Pin_1)
- net XD0: now also J4.23 (Pin_23)
- net XD1: now also J4.24 (Pin_24)
- net XD2: now also J4.25 (Pin_25)
- net XD3: now also J4.26 (Pin_26)
- net XD4: now also J4.27 (Pin_27)
- net XD5: now also J4.28 (Pin_28)
- net XD6: now also J4.29 (Pin_29)
- net XD7: now also J4.30 (Pin_30)
- net XE: now also J6.1 (Pin_1)
- net XIN: now also J5.2 (Pin_2)
- net XIRQ: now also J5.6 (Pin_6)
- net XRD: now also J5.7 (Pin_7)
- net XSLC: now also J5.4 (Pin_4)
- net XWR: now also J5.8 (Pin_8)
Other:
- moved on the sheet: D1, J1, J2, J3, J4, J5, R1

Commit message: about to delete extra silk
Parts:
- J6: value XE_LA -> XIN_LA
Connections:
- net XE: now also J5.2 (Pin_2); no longer J6.1 (Pin_1)
- net XIN: now also J6.1 (Pin_1); no longer J5.2 (Pin_2)
Changed lines of the file:
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@@
 		)
 	)
-	(label "XIN"
+	(label "XE"
 		(at 111.76 68.58 180)
 		(fields_autoplaced yes)
@@
 		)
 	)
-	(label "XE"
+	(label "XIN"
 		(at 86.36 54.61 0)
 		(fields_autoplaced yes)
@@
 			)
 		)
-		(property "Value" "XE_LA"
+		(property "Value" "XIN_LA"
 			(at 99.06 57.1499 0)
 			(effects

Commit message: dd adapter rev 1 ready to go to the fab
Parts:
- added TP1, TP2: TestPoint_Harwin, My Libraries:Harwin-S1751-46-Test-Point, symbol My Library:TestPoint_Harwin
Connections:
- net GND: now also TP1.1, TP2.1
Other:
- title: (none) -> CERBERUS 2100(tm) Digital Discovery(tm) Adapter
- moved on the sheet: D1, J1, J2, J3, J4, J5, J6, J7, R1
