File: One-to-One LA Adapter/One-to-One LA Adapter.kicad_pcb (KiCad board)
At the start: 2 copper layers, 32.5 x 62.9 mm, 6 parts, among them J1 Cerberus_Expansion, J2 Card_Header, J3 LA_Header, J4 XE_Header

Commit message: one-to-one rev1 ready for fab
Other:
- board text added: "GND"
- board text added: "cerberus 2100 1:1 LA adapter rev1, @baldengineer"
